File: MainBoard/USB3.sch (KiCad schematic (older format))
At the start: 15 parts

Commit message: partial redo of keyboard, invert differential pairs on USB conn
Parts:
- added U?: MX25L5121EMC-20G, SOP-8L_3P9X4P9_MAC, symbol MX25L5121EMC:MX25L5121EMC-20G
Connections:
- net +3V3: now also U?.7 (VCC)
- net GND: now also U?.8 (GND)
- net at U?.16 (SPISO): now also U?.3 (SO)
- net at U?.17 (SPICSB): now also U?.1 (CS#)
- net at U?.18 (SPISCK): now also U?.4 (SCLK)
- net at U?.19 (SPISI): now also U?.2 (SI)
- net at U?.35 (U3TXDP1): now also J?.9 (SSTX+); no longer J?.6 (SSRX+)
- net at U?.36 (U3TXDN1): now also J?.8 (SSTX-); no longer J?.5 (SSRX-)
- net at U?.38 (U3RXDP1): now also J?.6 (SSRX+); no longer J?.9 (SSTX+)
- net at U?.39 (U3RXDN1): now also J?.5 (SSRX-); no longer J?.8 (SSTX-)
- net at U?.52 (U3TXDP3): now also J?.9 (SSTX+); no longer J?.6 (SSRX+)
- net at U?.53 (U3TXDN3): now also J?.8 (SSTX-); no longer J?.5 (SSRX-)
- net at U?.55 (U3RXDP3): now also J?.6 (SSRX+); no longer J?.9 (SSTX+)
- net at U?.56 (U3RXDN3): now also J?.5 (SSRX-); no longer J?.8 (SSTX-)
- net at U?.11 (USB_SSTXP_DN2): now also J?.9 (SSTX+); no longer J?.6 (SSRX+)
- net at U?.12 (USB_SSTXM_DN2): now also J?.8 (SSTX-); no longer J?.5 (SSRX-)
- net at U?.14 (USB_SSRXP_DN2): now also J?.6 (SSRX+); no longer J?.9 (SSTX+)
- net at U?.15 (USB_SSRXM_DN2): now also J?.5 (SSRX-); no longer J?.8 (SSTX-)
- net at U?.19 (USB_SSTXP_DN3): now also J?.9 (SSTX+); no longer J?.6 (SSRX+)
- net at U?.20 (USB_SSTXM_DN3): now also J?.8 (SSTX-); no longer J?.5 (SSRX-)
- net at U?.22 (USB_SSRXP_DN3): now also J?.6 (SSRX+); no longer J?.9 (SSTX+)
- net at U?.23 (USB_SSRXM_DN3): now also J?.5 (SSRX-); no longer J?.8 (SSTX-)
- net at U?.26 (USB_SSTXP_DN4): now also J?.9 (SSTX+); no longer J?.6 (SSRX+)
- net at U?.27 (USB_SSTXM_DN4): now also J?.8 (SSTX-); no longer J?.5 (SSRX-)
- net at U?.29 (USB_SSRXP_DN4): now also J?.6 (SSRX+); no longer J?.9 (SSTX+)
- net at U?.3 (USB_SSTXP_DN1): now also J?.9 (SSTX+); no longer J?.6 (SSRX+)
- net at U?.30 (USB_SSRXM_DN4): now also J?.5 (SSRX-); no longer J?.8 (SSTX-)
- net at U?.4 (USB_SSTXM_DN1): now also J?.8 (SSTX-); no longer J?.5 (SSRX-)
- net at U?.6 (USB_SSRXP_DN1): now also J?.6 (SSRX+); no longer J?.9 (SSTX+)
- net at U?.7 (USB_SSRXM_DN1): now also J?.5 (SSRX-); no longer J?.8 (SSTX-)
Other:
- moved on the sheet: D?, J?, U?, Y?
