File: MainBoard/keyboard.sch (KiCad schematic (older format))
At the start: 101 parts, among them U2 ATmega32U4-AU

Commit message: mostly replace keyboard
Parts:
- added U3: CD74HC4067M, Package_SO:SOIC-24W_7.5x15.4mm_P1.27mm, symbol 74xx:CD74HC4067M
- SW1, SW10, SW100, SW11, SW12, SW13, SW14, SW15, SW16, SW17, SW18, SW19, SW2, SW20, SW21, SW22, SW23, SW24, SW25, SW26, SW27, SW28, SW29, SW3, SW30, SW31, SW32, SW33, SW34, SW35, SW36, SW37, SW38, SW39, SW4, SW40, SW41, SW42, SW43, SW44, SW45, SW46, SW47, SW48, SW49, SW5, SW50, SW51, SW52, SW53, SW54, SW55, SW56, SW57, SW58, SW59, SW6, SW60, SW61, SW62, SW63, SW64, SW65, SW66, SW67, SW68, SW69, SW7, SW70, SW71, SW72, SW73, SW74, SW75, SW76, SW77, SW78, SW79, SW8, SW80, SW81, SW82, SW83, SW84, SW85, SW86, SW87, SW88, SW89, SW9, SW90, SW91, SW92, SW93, SW94, SW95, SW96, SW97, SW98, SW99: renamed from SW?; footprint (none) -> Libs:Kailh_socket_PG1350
Connections:
- net at U2.1 (PE6): now also U3.13 (S3)
- net at U2.12 (PB7): now also SW28.3 (B), SW28.4 (B), SW29.3 (B), SW29.4 (B), SW30.3 (B), SW30.4 (B), SW31.3 (B), SW31.4 (B), SW32.3 (B), SW32.4 (B), SW33.3 (B), SW33.4 (B), SW34.3 (B), SW34.4 (B), SW35.3 (B), SW35.4 (B), SW36.3 (B), SW36.4 (B), SW37.3 (B), SW37.4 (B), SW38.3 (B), SW38.4 (B), SW39.3 (B), SW39.4 (B), SW40.3 (B), SW40.4 (B), SW41.3 (B), SW41.4 (B), SW42.3 (B), SW42.4 (B)
- net at U2.19 (PD1): now also U3.1 (COM)
- net at U2.25 (PD4): now also U3.10 (S0)
- net at U2.26 (PD6): now also SW43.3 (B), SW43.4 (B), SW44.3 (B), SW44.4 (B), SW45.3 (B), SW45.4 (B), SW46.3 (B), SW46.4 (B), SW47.3 (B), SW47.4 (B), SW48.3 (B), SW48.4 (B), SW49.3 (B), SW49.4 (B), SW50.3 (B), SW50.4 (B), SW51.3 (B), SW51.4 (B), SW52.3 (B), SW52.4 (B), SW53.3 (B), SW53.4 (B), SW54.3 (B), SW54.4 (B), SW55.3 (B), SW55.4 (B), SW56.3 (B), SW56.4 (B), SW57.3 (B), SW57.4 (B)
- net at U2.27 (PD7): now also U3.14 (S2)
- net at U2.28 (PB4): now also U3.15 (~E)
- net at U2.29 (PB5): now also SW1.3 (B), SW1.4 (B), SW10.3 (B), SW10.4 (B), SW11.3 (B), SW11.4 (B), SW2.3 (B), SW2.4 (B), SW3.3 (B), SW3.4 (B), SW4.3 (B), SW4.4 (B), SW5.3 (B), SW5.4 (B), SW6.3 (B), SW6.4 (B), SW7.3 (B), SW7.4 (B), SW8.3 (B), SW8.4 (B), SW9.3 (B), SW9.4 (B)
- net at U2.30 (PB6): now also SW12.3 (B), SW12.4 (B), SW13.3 (B), SW13.4 (B), SW14.3 (B), SW14.4 (B), SW15.3 (B), SW15.4 (B), SW16.3 (B), SW16.4 (B), SW17.3 (B), SW17.4 (B), SW18.3 (B), SW18.4 (B), SW19.3 (B), SW19.4 (B), SW20.3 (B), SW20.4 (B), SW21.3 (B), SW21.4 (B), SW22.3 (B), SW22.4 (B), SW23.3 (B), SW23.4 (B), SW24.3 (B), SW24.4 (B), SW25.3 (B), SW25.4 (B), SW26.3 (B), SW26.4 (B), SW27.3 (B), SW27.4 (B)
- net at U2.31 (PC6): now also U3.11 (S1)
- net at U2.32 (PC7): now also SW58.3 (B), SW58.4 (B), SW59.3 (B), SW59.4 (B), SW60.3 (B), SW60.4 (B), SW61.3 (B), SW61.4 (B), SW62.3 (B), SW62.4 (B), SW63.3 (B), SW63.4 (B), SW64.3 (B), SW64.4 (B), SW65.3 (B), SW65.4 (B), SW66.3 (B), SW66.4 (B), SW67.3 (B), SW67.4 (B), SW68.3 (B), SW68.4 (B), SW69.3 (B), SW69.4 (B), SW70.3 (B), SW70.4 (B), SW71.3 (B), SW71.4 (B), SW72.3 (B), SW72.4 (B)
- net at U2.36 (PF7): now also SW73.3 (B), SW73.4 (B), SW74.3 (B), SW74.4 (B), SW75.3 (B), SW75.4 (B), SW76.3 (B), SW76.4 (B), SW77.3 (B), SW77.4 (B), SW78.3 (B), SW78.4 (B), SW79.3 (B), SW79.4 (B), SW80.3 (B), SW80.4 (B), SW81.3 (B), SW81.4 (B), SW82.3 (B), SW82.4 (B), SW83.3 (B), SW83.4 (B), SW84.3 (B), SW84.4 (B), SW85.3 (B), SW85.4 (B), SW86.3 (B), SW86.4 (B), SW87.3 (B), SW87.4 (B)
- net at U2.37 (PF6): now also SW100.3 (B), SW100.4 (B), SW88.3 (B), SW88.4 (B), SW89.3 (B), SW89.4 (B), SW90.3 (B), SW90.4 (B), SW91.3 (B), SW91.4 (B), SW92.3 (B), SW92.4 (B), SW93.3 (B), SW93.4 (B), SW94.3 (B), SW94.4 (B), SW95.3 (B), SW95.4 (B), SW96.3 (B), SW96.4 (B), SW97.3 (B), SW97.4 (B), SW98.3 (B), SW98.4 (B), SW99.3 (B), SW99.4 (B)
- net at SW1.1 (A), SW1.2 (A), SW13.1 (A)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: now also U3.17 (I14)
- net at SW14.1 (A), SW14.2 (A), SW2.1 (A)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: now also U3.18 (I13)
- net at SW15.1 (A), SW15.2 (A), SW3.1 (A)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: now also U3.19 (I12)
- net at SW16.1 (A), SW16.2 (A), SW32.1 (A)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: now also U3.20 (I11)
- net at SW17.1 (A), SW17.2 (A), SW33.1 (A)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: now also U3.21 (I10)
- net at SW100.1 (A), SW100.2 (A), SW19.1 (A)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: now also U3.23 (I8)
- net at SW20.1 (A), SW20.2 (A), SW36.1 (A)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: now also U3.2 (I7)
- net at SW21.1 (A), SW21.2 (A), SW37.1 (A)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: now also U3.3 (I6)
- net at SW23.1 (A), SW23.2 (A), SW39.1 (A)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: now also U3.5 (I4)
- net at SW10.1 (A), SW10.2 (A), SW24.1 (A)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: now also U3.6 (I3)
- net at SW11.1 (A), SW11.2 (A), SW26.1 (A)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: now also U3.8 (I1)
- net at SW12.1 (A), SW12.2 (A), SW29.1 (A)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: now also U3.16 (I15)
- net at SW18.1 (A), SW18.2 (A), SW34.1 (A)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: now also U3.22 (I9)
- net at SW22.1 (A), SW22.2 (A), SW38.1 (A)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: now also U3.4 (I5)
- net at SW25.1 (A), SW25.2 (A), SW41.1 (A)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: now also U3.7 (I2)
- net at SW27.1 (A), SW27.2 (A), SW28.1 (A)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: now also SW57.1 (A), SW57.2 (A), SW72.1 (A), SW72.2 (A), SW86.1 (A), SW86.2 (A), SW93.1 (A), SW93.2 (A), U3.9 (I0)
Other:
- moved on the sheet: SW1, SW10, SW100, SW11, SW12, SW13, SW14, SW15, SW16, SW17, SW18, SW19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
